File: Design/KiCAD/AT89S52_Dev_Board.sch (KiCad schematic (older format))
At the start: 12 parts, among them J1 Jack-DC, J2 Conn_01x02, J3 VCC_12V, J4 VCC_5V, U1 L7812, U2 L7805

Commit message: modified
Parts:
- added C10, C11, C12, C9: CP, Capacitors_THT:C_Disc_D5.0mm_W2.5mm_P5.00mm, symbol CP
- added C6, C7, C8: C, Capacitors_THT:C_Disc_D5.0mm_W2.5mm_P5.00mm, symbol C
- added D2: LED, LEDs:LED_D3.0mm, symbol LED
- added J10: ISP, Socket_Strips:Socket_Strip_Straight_2x05_Pitch2.00mm, symbol Conn_02x05_Top_Bottom
- added J11: LCD Port, Socket_Strips:Socket_Strip_Straight_1x16_Pitch1.27mm, symbol Conn_01x16_Female
- added J5: Port 3, Socket_Strips:Socket_Strip_Straight_1x08_Pitch2.00mm, symbol Conn_01x08_Male
- added J6: Port 1, Socket_Strips:Socket_Strip_Straight_1x08_Pitch2.00mm, symbol Conn_01x08_Male
- added J7: Port 2, Socket_Strips:Socket_Strip_Straight_2x05_Pitch2.00mm, symbol Conn_01x08_Male
- added J8: Port 0, Socket_Strips:Socket_Strip_Straight_1x08_Pitch2.00mm, symbol Conn_01x08_Male
- added J9: Serial Port, Connectors_JST:JST_ZE_S09B-ZESK-2D_09x1.5mm_Angled, symbol DB9_Female
- added R1, R2: R, Resistors_THT:R_Axial_DIN0411_L9.9mm_D3.6mm_P15.24mm_Horizontal, symbol R
- added RV1: Contrast, Potentiometers:Potentiometer_Trimmer-EVM3E, symbol POT_TRIM
- added SW1: Reset, Buttons_Switches_THT:Push_E-Switch_KS01Q01, symbol SW_Push
- added SW2: SW_Push, Buttons_Switches_THT:Push_E-Switch_KS01Q01, symbol SW_Push
- added U3: AT89S52, Housings_DIP:DIP-40_W15.24mm, symbol AT89S52-RESCUE-AT89S52_Dev_Board
- added U4: MAX232, symbol MAX232
- added Y1: Crystal, Crystals:Resonator-2pin_w10.0mm_h5.0mm, symbol Crystal
Connections:
- net labels added: D3, D4, D5, D7
- wire segments 49 -> 248
Other:
- moved on the sheet: C2, C4, J3, U1

Commit message: modified
Connections:
- wire segments 248 -> 187

Commit message: modified
Parts:
- J2: value Conn_01x02 -> 12V AC
- J7: footprint Socket_Strips:Socket_Strip_Straight_2x05_Pitch2.00mm -> Socket_Strips:Socket_Strip_Straight_1x08_Pitch2.00mm
- R1, R2: footprint Resistors_THT:R_Axial_DIN0411_L9.9mm_D3.6mm_P15.24mm_Horizontal -> Resistors_THT:R_Axial_DIN0207_L6.3mm_D2.5mm_P7.62mm_Horizontal
- SW1, SW2: footprint Buttons_Switches_THT:Push_E-Switch_KS01Q01 -> Buttons_Switches_THT:SW_PUSH_6mm
- U1, U2: footprint TO_SOT_Packages_THT:TO-220-2_Horizontal -> TO_SOT_Packages_THT:TO-126_Vertical
- U4: footprint (none) -> Housings_DIP:DIP-16_W10.16mm
Connections:
- net labels added: D6, E, RS, RST, RXD, TXD
- net labels removed: D3, VCC_5V
- wire segments 187 -> 177
Other:
- moved on the sheet: C1, C2, C3, C4, C5, C8, D1, D2, J1, J10, J11, J2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
