File: Design/KiCAD/AT89S52_Dev_Board.kicad_pcb (KiCad board)
At the start: 2 copper layers, 120 x 75 mm, 12 parts, among them J1 Jack-DC, J2 Conn_01x02, J3 VCC_12V, J4 VCC_5V, U1 L7812, U2 L7805

Commit message: modified
Parts:
- added U3: AT89S52, Housings_DIP:DIP-40_W15.24mm, F.Cu at (86.0, 105.1)
Connections:
- C5 pad 1: +5V -> Net-(C5-Pad1)
- U2 pad 3: +5V -> Net-(C5-Pad1)
Routing:
- net Net-(C5-Pad1): track 0.00 -> 5.42 mm
- net +5V: track 23.2 -> 17.7 mm

Commit message: modified
Parts:
- added C10: CP, Capacitors_THT:C_Disc_D5.0mm_W2.5mm_P5.00mm, F.Cu at (34.5, 59.5)
- added C11: CP, Capacitors_THT:C_Disc_D5.0mm_W2.5mm_P5.00mm, F.Cu at (36.5, 78.0)
- added C12: CP, Capacitors_THT:C_Disc_D5.0mm_W2.5mm_P5.00mm, F.Cu at (45.0, 78.0)
- added C6: C, Capacitors_THT:C_Disc_D5.0mm_W2.5mm_P5.00mm, F.Cu at (144.0, 51.5)
- added C7: C, Capacitors_THT:C_Disc_D5.0mm_W2.5mm_P5.00mm, F.Cu at (144.0, 68.5)
- added C8: C, Capacitors_THT:C_Disc_D5.0mm_W2.5mm_P5.00mm, F.Cu at (108.5, 73.5)
- added C9: CP, Capacitors_THT:C_Disc_D5.0mm_W2.5mm_P5.00mm, F.Cu at (28.5, 77.5)
- added D2: LED, LEDs:LED_D3.0mm, F.Cu at (82.0, 79.0)
- added J10: ISP, Socket_Strips:Socket_Strip_Straight_2x05_Pitch2.00mm, F.Cu at (72.5, 87.5)
- added J11: LCD Port, Socket_Strips:Socket_Strip_Straight_1x16_Pitch1.27mm, F.Cu at (120.5, 35.0)
- added J5: Port 3, Socket_Strips:Socket_Strip_Straight_1x08_Pitch2.00mm, F.Cu at (122.0, 89.5)
- added J6: Port 1, Socket_Strips:Socket_Strip_Straight_1x08_Pitch2.00mm, F.Cu at (85.5, 89.0)
- added J7: Port 2, Socket_Strips:Socket_Strip_Straight_1x08_Pitch2.00mm, F.Cu at (141.5, 37.0)
- added J8: Port 0, Socket_Strips:Socket_Strip_Straight_1x08_Pitch2.00mm, F.Cu at (85.5, 20.0)
- added J9: Serial Port, Connectors_JST:JST_ZE_S09B-ZESK-2D_09x1.5mm_Angled, F.Cu at (29.5, 82.0)
- added R1: R, Resistors_THT:R_Axial_DIN0207_L6.3mm_D2.5mm_P7.62mm_Horizontal, F.Cu at (108.0, 69.5)
- added R2: R, Resistors_THT:R_Axial_DIN0207_L6.3mm_D2.5mm_P7.62mm_Horizontal, F.Cu at (83.5, 65.0)
- added RV1: Contrast, Potentiometers:Potentiometer_Trimmer-EVM3E, F.Cu at (123.0, 22.0)
- added SW1: Reset, Buttons_Switches_THT:SW_PUSH_6mm, F.Cu at (121.0, 72.0)
- added SW2: SW_Push, Buttons_Switches_THT:SW_PUSH_6mm, F.Cu at (93.0, 74.0)
- added U4: MAX232, Housings_DIP:DIP-16_W10.16mm, F.Cu at (29.0, 73.5)
- added Y1: Crystal, Crystals:Resonator-2pin_w10.0mm_h5.0mm, F.Cu at (141.5, 57.5)
- C1: footprint Capacitors_THT:CP_Radial_Tantal_D8.0mm_P5.00mm -> Capacitors_THT:CP_Radial_D8.0mm_P5.00mm
- C2: footprint Capacitors_THT:C_Disc_D3.0mm_W2.0mm_P2.50mm -> Capacitors_THT:C_Disc_D5.0mm_W2.5mm_P5.00mm
- C3, C4, C5: footprint Capacitors_THT:C_Disc_D3.0mm_W2.0mm_P2.50mm -> Capacitors_THT:C_Disc_D5.0mm_W2.5mm_P2.50mm
- J2: value Conn_01x02 -> 12V AC
- U1, U2: footprint TO_SOT_Packages_THT:TO-220-3_Horizontal -> TO_SOT_Packages_THT:TO-220-2_Horizontal
- moved U3 47.2 mm to (83.0, 58.0), turned to 90 degrees
- moved C1 4.03 mm to (33.0, 35.5)
- moved C2 4.03 mm to (62.5, 43.0)
- moved C3 4.03 mm to (49.5, 43.0)
- moved C4 4.03 mm to (55.5, 43.0)
- moved C5 4.03 mm to (70.5, 43.0)
- moved D1 4.03 mm to (36.0, 48.5)
- moved J1 4.03 mm to (41.5, 23.0)
- moved J2 4.03 mm to (28.5, 47.0)
- moved J3 4.03 mm to (81.0, 19.6)
- moved J4 4.03 mm to (75.6, 19.6)
- moved U1 4.03 mm to (50.5, 38.0)
- moved U2 4.03 mm to (63.5, 38.0)
Connections:
- C5 pad 1: Net-(C5-Pad1) -> +5V
- U3 pad 1: Net-(U3-Pad1) -> /RS
- U3 pad 10: Net-(U3-Pad10) -> /RXD
- U3 pad 11: Net-(U3-Pad11) -> /TXD
- U3 pad 2: Net-(U3-Pad2) -> /E
- U3 pad 20: Net-(U3-Pad20) -> GND
- U3 pad 31: Net-(U3-Pad31) -> +5V
- U3 pad 40: Net-(U3-Pad40) -> +5V
- U3 pad 5: Net-(U3-Pad5) -> /D4
- U3 pad 6: Net-(U3-Pad6) -> /D5
- U3 pad 7: Net-(U3-Pad7) -> /D6
- U3 pad 8: Net-(U3-Pad8) -> /D7
- U3 pad 9: Net-(U3-Pad9) -> /RST
Routing:
- net GND: track 110.2 -> 153.2 mm
- net +12V: track 57.3 -> 22.0 mm
- net Net-(C5-Pad1): track 5.42 -> 0.00 mm
- net +5V: track 17.7 -> 15.5 mm

Commit message: modified
Parts:
- moved RV1 75.0 mm to (72.5, 77.5)
- moved J11 69.8 mm to (74.0, 87.0)
- moved J5 34.7 mm to (126.0, 55.0)
- moved C10 28.9 mm to (63.0, 54.5)
- moved Y1 22.5 mm to (140.0, 35.0)
- moved J10 20.8 mm to (64.0, 68.5)
- moved J7 19.7 mm to (131.5, 20.0), turned to 270 degrees
- moved R2 18.3 mm to (80.0, 47.0)
- moved D2 18.0 mm to (78.0, 61.5)
- moved C7 16.0 mm to (140.0, 53.0)
- moved SW1 15.0 mm to (136.0, 73.0), turned to 180 degrees
- moved C9 13.0 mm to (28.5, 64.5), turned to 90 degrees
- moved U3 11.9 mm to (86.0, 46.5)
- moved SW2 11.5 mm to (81.5, 73.0)
- moved C8 10.0 mm to (118.5, 73.5)
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